Commit message: Rescaled body segments to fit data set better

File: urdf/mannequin_two_arms.urdf (robot description, URDF)
Before this commit: robot mannequin, 14 links, 13 joints
Links:
- link body_link: geometry collision cylinder length=0.1 radius=0.2; visual mesh filename=package://mannequin/models/mannequin/meshes/body_formatted.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
- link left_hand_link: geometry collision box size=0.03 0.01 0.05; visual mesh filename=package://mannequin/models/mannequin/meshes/hand_formatted.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
- link lower_left_arm_link: geometry collision cylinder length=0.3 radius=0.03; visual mesh filename=package://mannequin/models/mannequin/meshes/lower_arm_forma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
- link lower_right_arm_link: geometry collision cylinder length=0.3 radius=0.03; visual mesh filename=package://mannequin/models/mannequin/meshes/lower_arm_forma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
- link right_hand_link: geometry collision box size=0.03 0.01 0.05; visual mesh filename=package://mannequin/models/mannequin/meshes/hand_formatted.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
- link upper_left_arm_link: geometry collision cylinder length=0.3 radius=0.03; visual mesh filename=package://mannequin/models/mannequin/meshes/upper_arm_forma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
- link upper_right_arm_link: geometry collision cylinder length=0.3 radius=0.03; visual mesh filename=package://mannequin/models/mannequin/meshes/upper_arm_forma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

Commit message: Small edit to unify two arms and full

File: urdf/mannequin_two_arms.urdf (robot description, URDF)
Before this commit: robot mannequin, 14 links, 13 joints
Joints:
- joint left_elbow_joint: limit lower=0.01 upper=3.0 effort=1 velocity=0.5 -> lower=0.01 upper=3.0 effort=100 velocity=0.5
- joint left_shoulder_pitch_joint: limit lower=-1.57 upper=0 effort=4 velocity=0.5 -> lower=-1.57 upper=0 effort=100 velocity=0.5
- joint left_shoulder_yaw_joint: limit lower=-1.1 upper=1.5 effort=1 velocity=0.5 -> lower=-1.1 upper=1.5 effort=100 velocity=0.5
- joint right_elbow_joint: limit lower=0.01 upper=3.0 effort=1 velocity=0.5 -> lower=0.01 upper=3.0 effort=100 velocity=0.5
- joint right_shoulder_pitch_joint: limit lower=0 upper=1.57 effort=4 velocity=0.5 -> lower=0 upper=1.57 effort=100 velocity=0.5
- joint right_shoulder_yaw_joint: limit lower=-1.5 upper=1.1 effort=1 velocity=0.5 -> lower=-1.5 upper=1.1 effort=100 velocity=0.5
