Commit message: final tweaks

File: urdf/mannequin_fully_articulated.urdf.xacro (robot description, xacro)
@@ -8,10 +8,12 @@
         </plugin>
     </gazebo>
+    <xacro:property name="joint_effort" value="100"/>
+    <xacro:property name="joint_velocity" value="0.5"/>
     <!-- * * * Link Definitions * * * -->
-    <link name="base_link"> <!-- Base link is used to allow all body parts to have inertial settings -->
+    <link name="base_link"> <!-- Base link allows the body to "float"-->
         <visual>
-            <origin rpy="0.1 0 0" xyz="0 0 0"/>
-            <geometry>
-                <box size="0.1 0.1 1"/>
+            <origin rpy="0 0 0" xyz="0 0 0"/>
+            <geometry>
+                <cylinder radius="0.6" length="0.03"/>
             </geometry>
         </visual>
@@ -19,11 +21,11 @@
             <origin xyz="0 0 0" rpy="0 0 0"/>
             <geometry>
-                <box size="0.5 0.5 1"/>
+                <cylinder radius="0.6" length="0.03"/>
             </geometry>
         </collision>
 	</link>
     <gazebo reference="base_link">
-        <kp>10000.0</kp>
-        <kd>10000.0</kd>
+        <kp>50000.0</kp>
+        <kd>50000.0</kd>
         <mu1>10.0</mu1>
         <mu2>10.0</mu2>
@@ -45,5 +47,5 @@
         </collision>
         <inertial>
-            <origin xyz="0 0 0.145" rpy="0 0 0"/>
+            <origin xyz="0 0 0.145" rpy="-0.01 0 0"/>
             <mass value="15.3" />
             <inertia ixx="0.2913375" ixy="0.0" ixz="0.0" iyy="0.162920775" iyz="0.0" izz="0.239803275"/>
@@ -78,6 +80,33 @@
 	</link>
     <gazebo reference="upper_body_link">
-        <kp>5000.0</kp>
-        <kd>5000.0</kd>
+        <kp>10000.0</kp>
+        <kd>10000.0</kd>
+        <mu1>10.0</mu1>
+        <mu2>10.0</mu2>
+        <material>Gazebo/White</material>
+    </gazebo>
+    <link name="head_link">
+    	<visual>
+            <origin rpy="0.0 0 0" xyz="0 0 0"/>
+            <geometry>
+                <!-- Material color set to white in blender -->
+                <mesh filename="package://mannequin/models/mannequin/meshes/head_formatted.dae"/>
+            </geometry>
+        </visual>
+        <collision>
+            <origin xyz="0 0 0.073" rpy="0 0 0"/>
+            <geometry>
+                <sphere radius="0.073"/>
+            </geometry>
+        </collision>
+        <inertial>
+            <origin xyz="0 0 0.073" rpy="0 0 0"/>
+            <mass value="4.7" />
+            <inertia ixx="0.01001852" ixy="0.0" ixz="0.0" iyy="0.01001852" iyz="0.0" izz="0.01001852"/>
+        </inertial>
+	</link>
+    <gazebo reference="head_link">
+        <kp>10000.0</kp>
+        <kd>10000.0</kd>
         <mu1>10.0</mu1>
         <mu2>10.0</mu2>
@@ -88,18 +117,47 @@
     	<parent link="base_link"/>
         <child link="lower_body_link"/>
+        <origin xyz="0 0 1" rpy="0 0 0"/>
     </joint>
     <joint name="torso_mid_joint" type="revolute">
+	    <hardwareInterface>hardware_interface/EffortJointInterface</hardwareInterface>
         <parent link="lower_body_link"/>
         <child link="upper_body_link"/>
         <axis xyz="1 0 0"/> <!-- As is, the mannequin torso can only bend side to side, as this is what I have ROM data on-->
-        <limit lower="-0.611" upper="0.611" effort="2" velocity="1.0"/>
-        <origin xyz="0 0.01 0.207" rpy="0 0 0"/>
+        <limit lower="-0.611" upper="0.611" effort="1000" velocity="${joint_velocity}"/>
+        <origin xyz="0 0 0.260" rpy="0 0 0"/>
     </joint>
+    <joint name="neck_joint" type="revolute">
+	    <hardwareInterface>hardware_interface/EffortJointInterface</hardwareInterface>
+        <parent link="upper_body_link"/>
+        <child link="head_link"/>
+        <axis xyz="1 0 0"/> <!-- As is, the mannequin head can only tilt left/right to simplify the joint-->
+        <limit lower="-0.785" upper="0.785" effort="${joint_effort}" velocity="${joint_velocity}"/>
+        <origin xyz="0 0.0 0.358" rpy="0 0 0"/>
+    </joint>
+    <transmission name="torsotran">
+	    <type>transmission_interface/SimpleTransmission</type>
+		<joint name="torso_mid_joint">
+	        <hardwareInterface>hardware_interface/EffortJointInterface</hardwareInterface>
+	    </joint>
+		<actuator name="torsomotor">
+	        <mechanicalReduction>50</mechanicalReduction>
+	    </actuator>
+	</transmission>
+	<transmission name="necktran">
+	    <type>transmission_interface/SimpleTransmission</type>
+		<joint name="neck_joint">
+	        <hardwareInterface>hardware_interface/EffortJointInterface</hardwareInterface>
+	    </joint>
+		<actuator name="headmotor">
+	        <mechanicalReduction>50</mechanicalReduction>
+	    </actuator>
+	</transmission>
     <!-- Macro and variables for creating the arms -->
     <xacro:property name="pseudo_radius" value="0.01"/>
     <xacro:property name="pseudo_mass" value="0.01"/>
     <xacro:property name="pseudo_I" value="4e-07"/>
-    <xacro:property name="arm_vertical_offset" value="0.287"/>
-    <xacro:property name="arm_horizontal_offset" value="0.152"/>
+    <xacro:property name="arm_vertical_offset" value="0.23"/>
+    <xacro:property name="upper_arm_horizontal_offset" value="0.17"/>
+    <xacro:property name="lower_arm_horizontal_offset" value="0.34"/>
     <xacro:macro name="arm" params="side reflection">
     	<!-- Shoulder and upper arm definitions-->
@@ -119,6 +177,6 @@
     	</link>
     	<gazebo reference="${side}_shoulder_roll_link">
-		    <kp>1000.0</kp>
-		    <kd>1000.0</kd>
+		    <kp>10000.0</kp>
+		    <kd>10000.0</kd>
 		    <mu1>10.0</mu1>
 		    <mu2>10.0</mu2>
@@ -139,6 +197,6 @@
     	</link>
     	<gazebo reference="${side}_shoulder_pitch_link">
-		    <kp>1000.0</kp>
-		    <kd>1000.0</kd>
+		    <kp>10000.0</kp>
+		    <kd>10000.0</kd>
 		    <mu1>10.0</mu1>
 		    <mu2>10.0</mu2>
@@ -159,6 +217,6 @@
     	</link>
     	<gazebo reference="${side}_shoulder_yaw_link">
-		    <kp>1000.0</kp>
-		    <kd>1000.0</kd>
+		    <kp>10000.0</kp>
+		    <kd>10000.0</kd>
 		    <mu1>10.0</mu1>
 		    <mu2>10.0</mu2>
@@ -193,22 +251,25 @@
 		</gazebo>
 		<joint name="${side}_shoulder_roll_joint" type="revolute">
+	        <hardwareInterface>hardware_interface/EffortJointInterface</hardwareInterface>
 		    <parent link="upper_body_link"/>
 		    <child link="${side}_shoulder_roll_link"/>
-		    <axis xyz="1 0 0"/>
-		    <limit lower="-1.05" upper="3.14" effort="2" velocity="1.0"/>
-		    <origin xyz="0 ${arm_horizontal_offset * reflection} ${arm_vertical_offset}" rpy="0 0 0"/>
+		    <axis xyz="${reflection} 0 0"/>
+		    <limit lower="-1.05" upper="3.14" effort="${joint_effort}" velocity="${joint_velocity}"/>
+		    <origin xyz="-.02 ${upper_arm_horizontal_offset * reflection} ${arm_vertical_offset}" rpy="0 0 0"/>
 		</joint>
 		<joint name="${side}_shoulder_pitch_joint" type="revolute">
+	        <hardwareInterface>hardware_interface/EffortJointInterface</hardwareInterface>
 		    <parent link="${side}_shoulder_roll_link"/>
 		    <child link="${side}_shoulder_pitch_link"/>
-		    <axis xyz="0 ${reflection} 0"/>
-		    <limit lower="-1.3" upper="3.14" effort="2" velocity="1.0"/>
+		    <axis xyz="0 1 0"/>
+		    <limit lower="-1.3" upper="3.14" effort="${joint_effort}" velocity="${joint_velocity}"/>
 		    <origin xyz="0 0 0" rpy="0 0 0"/>
 		</joint>
 		<joint name="${side}_shoulder_yaw_joint" type="revolute">
+	        <hardwareInterface>hardware_interface/EffortJointInterface</hardwareInterface>
 		    <parent link="${side}_shoulder_pitch_link"/>
 		    <child link="${side}_shoulder_yaw_link"/>
-		    <axis xyz="0 0 ${reflection}"/>
-		    <limit lower="-1.0" upper="1.5" effort="2" velocity="1.0"/>
+		    <axis xyz="0 0 ${-1*reflection}"/>
+		    <limit lower="-1.0" upper="1.5" effort="${joint_effort}" velocity="${joint_velocity}"/>
 		    <origin xyz="0 0 0" rpy="0 0 0"/>
 		</joint>
@@ -216,4 +277,5 @@
 		    <parent link="${side}_shoulder_yaw_link"/>
 		    <child link="${side}_upper_arm_link"/>
+		    <origin xyz="0 0 0" rpy="0 0 0"/>
 		</joint>
 		<!-- "Invisible" links for DOF of the elbow (flexion/extension[-0.17,2.62] and supination/pronation[-1.40,1.40]) -->
@@ -269,5 +331,5 @@
 		        <origin xyz="0 0 -0.128" rpy="0 0 0"/>
 		        <geometry>
-		            <cylinder radius="0.035" length="0.256"/>
+		            <cylinder radius="0.035" length="0.25"/>
 		        </geometry>
 		    </collision>
@@ -286,15 +348,18 @@
 		</gazebo>
 		<joint name="${side}_elbow_flexion_joint" type="revolute">
+	        <hardwareInterface>hardware_interface/EffortJointInterface</hardwareInterface>
 		    <parent link="${side}_upper_arm_link"/>
 		    <child link="${side}_elbow_flexion_link"/>
-		    <axis xyz="1 0 0"/>
-		    <limit lower="-1.05" upper="3.14" effort="2" velocity="1.0"/>
-		    <origin xyz="0 0 ${-1 * arm_vertical_offset}" rpy="0 0 0"/>
+		    <axis xyz="0 -1 0"/>
+		    <limit lower="-1.05" upper="3.14" effort="50" velocity="${joint_velocity}"/>
+		    <origin xyz="0 0 ${-1 * lower_arm_horizontal_offset}" rpy="0 0 0"/>
 		</joint>
 		<joint name="${side}_elbow_pronation_joint" type="revolute">
+	        <hardwareInterface>hardware_interface/EffortJointInterface</hardwareInterface>
 		    <parent link="${side}_elbow_flexion_link"/>
 		    <child link="${side}_elbow_pronation_link"/>
-		    <axis xyz="0 ${reflection} 0"/>
-		    <limit lower="-1.3" upper="3.14" effort="2" velocity="1.0"/>
+		    <axis xyz="0 0 ${reflection}"/>
+		    <limit lower="-1.3" upper="3.14" effort="50" velocity="${joint_velocity}"/>
+	        <hardwareInterface>hardware_interface/EffortJointInterface</hardwareInterface>
 		    <origin xyz="0 0 0" rpy="0 0 0"/>
 		</joint>
@@ -354,5 +419,5 @@
 		    </visual>
 		    <collision>
-		        <origin xyz="0 0 0" rpy="0 0 0"/>
+		        <origin xyz="0 0 -0.092" rpy="0 0 0"/>
 		        <geometry>
 		            <box size="0.077 0.028 0.184"/>
@@ -373,20 +438,23 @@
 		</gazebo>
 		<joint name="${side}_wrist_flexion_joint" type="revolute">
+	        <hardwareInterface>hardware_interface/EffortJointInterface</hardwareInterface>
 		    <parent link="${side}_lower_arm_link"/>
 		    <child link="${side}_wrist_flexion_link"/>
 		    <axis xyz="1 0 0"/>
-		    <limit lower="-1.05" upper="3.14" effort="2" velocity="1.0"/>
-		    <origin xyz="0 0 -${arm_vertical_offset - 0.05}" rpy="0 0 0"/>
+		    <limit lower="-1.396" upper="1.22" effort="5" velocity="${joint_velocity}"/>
+		    <origin xyz="0 0 -0.25" rpy="0 0 0"/>
 		</joint>
 		<joint name="${side}_wrist_deviation_joint" type="revolute">
+	        <hardwareInterface>hardware_interface/EffortJointInterface</hardwareInterface>
 		    <parent link="${side}_wrist_flexion_link"/>
 		    <child link="${side}_wrist_deviation_link"/>
 		    <axis xyz="0 ${reflection} 0"/>
-		    <limit lower="-1.3" upper="3.14" effort="2" velocity="1.0"/>
-		    <origin xyz="0 0 0" rpy="0 0 0"/>
+		    <limit lower="-0.523" upper="0.349" effort="5" velocity="${joint_velocity}"/>
+		    <origin xyz="0 ${reflection*0.01} 0" rpy="0 0 0"/>
 		</joint>
 		<joint name="${side}_hand_joint" type="fixed">
 		    <parent link="${side}_wrist_deviation_link"/>
 		    <child link="${side}_hand_link"/>
+		    <origin xyz="0 0 0" rpy="0 0 ${1.57*reflection}"/>
 		</joint>
     	<!-- ***** Actuator Definitions for arm ***** -->
@@ -398,6 +466,5 @@
 		    </joint>
 		    <actuator name="${side}shoulderrollmotor">
-		        <hardwareInterface>hardware_interface/EffortJointInterface</hardwareInterface>
-		        <mechanicalReduction>1</mechanicalReduction>
+		        <mechanicalReduction>50</mechanicalReduction>
 		    </actuator>
 		</transmission>
@@ -408,6 +475,5 @@
 		    </joint>
 		    <actuator name="${side}shoulderpitchmotor">
-		        <hardwareInterface>hardware_interface/EffortJointInterface</hardwareInterface>
-		        <mechanicalReduction>1</mechanicalReduction>
+		        <mechanicalReduction>50</mechanicalReduction>
 		    </actuator>
 		</transmission>
@@ -418,6 +484,5 @@
 		    </joint>
 		    <actuator name="${side}shoulderyawmotor">
-		        <hardwareInterface>hardware_interface/EffortJointInterface</hardwareInterface>
-		        <mechanicalReduction>1</mechanicalReduction>
+		        <mechanicalReduction>50</mechanicalReduction>
 		    </actuator>
 		</transmission>
@@ -429,6 +494,5 @@
 		    </joint>
 		    <actuator name="${side}elbowflexionmotor">
-		        <hardwareInterface>hardware_interface/EffortJointInterface</hardwareInterface>
-		        <mechanicalReduction>1</mechanicalReduction>
+		        <mechanicalReduction>50</mechanicalReduction>
 		    </actuator>
 		</transmission>
@@ -439,6 +503,5 @@
 		    </joint>
 		    <actuator name="${side}elbowpronationmotor">
-		        <hardwareInterface>hardware_interface/EffortJointInterface</hardwareInterface>
-		        <mechanicalReduction>1</mechanicalReduction>
+		        <mechanicalReduction>50</mechanicalReduction>
 		    </actuator>
 		</transmission>
@@ -450,6 +513,5 @@
 		    </joint>
 		    <actuator name="${side}wristflexionmotor">
-		        <hardwareInterface>hardware_interface/EffortJointInterface</hardwareInterface>
-		        <mechanicalReduction>1</mechanicalReduction>
+		        <mechanicalReduction>50</mechanicalReduction>
 		    </actuator>
 		</transmission>
@@ -460,6 +522,5 @@
 		    </joint>
 		    <actuator name="${side}wristdeviationmotor">
-		        <hardwareInterface>hardware_interface/EffortJointInterface</hardwareInterface>
-		        <mechanicalReduction>1</mechanicalReduction>
+		        <mechanicalReduction>50</mechanicalReduction>
 		    </actuator>
 		</transmission>
@@ -467,3 +528,145 @@
     <xacro:arm side="left" reflection="1"/>
     <xacro:arm side="right" reflection="-1"/>
+    <xacro:property name="leg_joint_effort" value="2000"/> <!-- The legs have to support the whole body, so they need high effort cap -->
+    <xacro:property name="leg_joint_velocity" value="2.0"/>
+    <xacro:macro name="leg" params="side reflection">
+    	<link name="${side}_thigh_link">
+    		<visual>
+		        <origin rpy="0.0 0 0" xyz="0 0 0"/>
+		        <geometry>
+		            <!-- Material color set to white in blender -->
+		            <mesh filename="package://mannequin/models/mannequin/meshes/upper_leg_formatted.dae"/>
+		        </geometry>
+		    </visual>
+		    <collision>
+		        <origin xyz="0 0 -0.240" rpy="0 0 0"/>
+		        <geometry>
+		            <cylinder radius="0.095" length=".475"/>
+		        </geometry>
+		    </collision>
+		    <inertial>
+		        <origin xyz="0 0 -0.240" rpy="0 0 0"/>
+		        <mass value="7.4" />
+		        <inertia ixx="0.15877625" ixy="0.0" ixz="0.0" iyy="0.15877625" iyz="0.0" izz="0.0333925"/>
+		    </inertial>
+		</link>
+		<gazebo reference="${side}_thigh_link">
+		    <kp>5000.0</kp>
+		    <kd>5000.0</kd>
+		    <mu1>10.0</mu1>
+		    <mu2>10.0</mu2>
+		    <material>Gazebo/White</material>
+		</gazebo>
+		<link name="${side}_calf_link">
+			<visual>
+		        <origin rpy="0.0 0 0" xyz="0 0 0"/>
+		        <geometry>
+		            <!-- Material color set to white in blender -->
+		            <mesh filename="package://mannequin/models/mannequin/meshes/lower_leg_formatted.dae"/>
+		        </geometry>
+		    </visual>
+		    <collision>
+		        <origin xyz="0 0 -0.217" rpy="0 0 0"/>
+		        <geometry>
+		            <cylinder radius="0.056" length=".433"/>
+		        </geometry>
+		    </collision>
+		    <inertial>
+		        <origin xyz="0 0 -0.217" rpy="0 0 0"/>
+		        <mass value="2.9" />
+		        <inertia ixx="0.0475834416667" ixy="0.0" ixz="0.0" iyy="0.0475834416667" iyz="0.0" izz="0.0045472"/>
+		    </inertial>
+		</link>
+		<gazebo reference="${side}_calf_link">
+		    <kp>5000.0</kp>
+		    <kd>5000.0</kd>
+		    <mu1>10.0</mu1>
+		    <mu2>10.0</mu2>
+		    <material>Gazebo/White</material>
+		</gazebo>
+		<link name="${side}_foot_link">
+			<visual>
+		        <origin rpy="0.0 0 0" xyz="0 0 0"/>
+		        <geometry>
+		            <!-- Material color set to white in blender -->
+		            <mesh filename="package://mannequin/models/mannequin/meshes/foot_formatted.dae"/>
+		        </geometry>
+		    </visual>
+		    <collision>
+		        <origin xyz="0.1205 0.0445 -0.014" rpy="0 0 0"/>
+		        <geometry>
+		        	<!--w=0.089 d=.028 h=0.241-->
+		            <box size="0.241 0.089 0.028"/>
+		        </geometry>
+		    </collision>
+		    <inertial>
+		        <origin xyz="0.1205 0.0445 -0.014" rpy="0 0 0"/>
+		        <mass value="1.2" /> <!--Iw = 0.0058865, Id = 0.0066002, Ih = 0.0008705-->
+		        <inertia ixx="0.0008705" ixy="0.0" ixz="0.0" iyy="0.0058865" iyz="0.0" izz="0.0066002"/>
+		    </inertial>
+		</link>
+		<gazebo reference="${side}_foot_link">
+		    <kp>5000.0</kp>
+		    <kd>5000.0</kd>
+		    <mu1>10.0</mu1>
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